File: charging_station/KiCad/PIHAT/PIHAT.kicad_pcb (KiCad board)
At the start: 2 copper layers, 135 x 56 mm, 32 parts, among them J1 GPIO, J2 5v(Vin), J3 WD_F, J4 Raspberry Control Signals, J5 RFID1, J6 RFID2, J7 MPPT, J8 PS, J9 RFID3, Q1 AO3400A, Q10 AO3401A, Q4 AO3401A, Q5 AO3400A, Q6 AO3401A, Q7 AO3400A, Q8 AO3401A, Q9 AO3400A, SW2 Sw_1, SW6 Sw_1, SW7 Sw_1, U2 TPS3430WDRC, U3 IM03GR, U4 TLV809EA29DBZR

Commit message: cd: hat: finalized schematic + rough layout
Parts:
- removed the J7 at (195.4, 39.3)
- removed the J8 at (204.5, 39.3)
- removed Q10: AO3401A, Package_TO_SOT_SMD:SOT-23
- removed Q9: AO3400A, Package_TO_SOT_SMD:SOT-23
- removed SW2, SW6, SW7: Sw_1, Button_Switch_SMD:SW_SPDT_CK_JS102011SAQN
- added H1: MountingHole, MountingHole:MountingHole_2.2mm_M2_DIN965, F.Cu at (238.2, 159.2)
- added H2: MountingHole, MountingHole:MountingHole_2.5mm, F.Cu at (277.4, 142.4)
- added J2: MPPT, TerminalBlock_Phoenix:TerminalBlock_Phoenix_PT-1,5-2-3.5-H_1x02_P3.50mm_Horizontal, F.Cu at (262.8, 132.7)
- added J3: PS, TerminalBlock_Phoenix:TerminalBlock_Phoenix_PT-1,5-2-3.5-H_1x02_P3.50mm_Horizontal, F.Cu at (272.4, 132.7)
- added Q2: AO3400A, Package_TO_SOT_SMD:SOT-23, F.Cu at (222.2, 72.1)
- added Q3: AO3401A, Package_TO_SOT_SMD:SOT-23, F.Cu at (227.2, 67.7)
- added U1: MSK12C02G25-B, external_ECAD:SW-SMD_MSK12C02G25-B, F.Cu at (223.2, 129.4)
- added U6: TLV809EA29DBZR, external_ECAD:SOT-23-3_L2.9-W1.3-P0.95-LS2.4-BR, F.Cu at (231.3, 79.4)
- added U7: TPS3430WDRC, Package_SON:VSON-10-1EP_3x3mm_P0.5mm_EP1.65x2.4mm, F.Cu at (217.4, 91.4)
- C2: value C_Small -> 100nF; footprint Capacitor_SMD:C_0805_2012Metric_Pad1.18x1.45mm_HandSolder -> Capacitor_SMD:C_0603_1608Metric
- C3: value 100nF -> C_Small; footprint Capacitor_SMD:C_0603_1608Metric -> Capacitor_SMD:C_0805_2012Metric_Pad1.18x1.45mm_HandSolder
- C4: value 100nF -> 1nF
- C5: value 1nF -> 100nF
- J9: renamed from J1; moved to F.Cu
- MH1, MH2, MH3, MH4: moved to B.Cu
- Q1, Q7: value AO3400A -> AO3401A
- Q6, Q8: value AO3401A -> AO3400A
- U2: value TPS3430WDRC -> MSK12C02G25-B; footprint Package_SON:VSON-10-1EP_3x3mm_P0.5mm_EP1.65x2.4mm -> external_ECAD:SW-SMD_MSK12C02G25-B
- U3: value IM03GR -> MSK12C02G25-B; footprint external_ECAD:RELAY-SMD_IMXXGR -> external_ECAD:SW-SMD_MSK12C02G25-B
- U4: value TLV809EA29DBZR -> IM03GR; footprint external_ECAD:SOT-23-3_L2.9-W1.3-P0.95-LS2.4-BR -> external_ECAD:RELAY-SMD_IMXXGR
- moved J8 150.7 mm to (247.3, 177.2)
- moved J7 149.1 mm to (260.8, 172.4)
- moved U4 121.2 mm to (251.0, 167.4)
- moved J1 120.4 mm to (221.7, 151.2), turned to 90 degrees
- moved J4 111.3 mm to (164.5, 172.5)
- moved MH2 99.5 mm to (155.5, 130.4), turned to 180 degrees
- moved MH4 99.5 mm to (155.5, 179.4), turned to 180 degrees
- moved J5 97.6 mm to (189.5, 172.5)
- moved J6 94.3 mm to (222.0, 172.5)
- moved U3 92.2 mm to (248.2, 129.4)
- moved D1 91.5 mm to (243.3, 167.2), turned to 90 degrees
- moved U2 84.3 mm to (235.7, 129.4)
- moved C3 46.3 mm to (207.3, 91.0)
- moved Q5 32.5 mm to (232.1, 67.7)
- moved Q7 32.5 mm to (237.0, 67.7)
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- renumbered J2 to J1, J5 to J4, J6 to J5, J9 to J6, J4 to J7, J3 to J8
Connections:
- C2 pad 1: Net-(U2-CWD) -> +3.3V
- C3 pad 1: +3.3V -> Net-(U7-CWD)
- C4 pad 1: +3.3V -> Net-(Q6-D)
- C5 pad 1: Net-(Q9-D) -> +3.3V
- J1 pad 1: GND -> +5V
- J1 pad 2: +5V -> GND
- J8 pad 1: Net-(J3-Pin_1) -> Net-(J8-Pin_1)
- J8 pad 2: Net-(J3-Pin_2) -> Net-(J8-Pin_2)
- Q1 pad 2: GND -> +3.3V
- Q1 pad 3: /Watchdog/WD_FAULT -> /Watchdog/SET0
- Q4 pad 1: Net-(Q4-G) -> /Watchdog/SET0
- Q4 pad 3: /Watchdog/SET0 -> Net-(D2-K)
- Q5 pad 1: Net-(Q4-G) -> /Watchdog/SET0
- Q5 pad 3: /Watchdog/SET0 -> Net-(D2-K)
- Q6 pad 1: /Watchdog/SET0 -> Net-(Q6-G)
- Q6 pad 2: +3.3V -> GND
- Q6 pad 3: Net-(D2-K) -> Net-(Q6-D)
- Q7 pad 1: /Watchdog/SET0 -> Net-(Q7-G)
- Q7 pad 2: GND -> +3.3V
- Q7 pad 3: Net-(D2-K) -> Net-(Q6-G)
- Q8 pad 2: +3.3V -> GND
- Q8 pad 3: Net-(Q8-D) -> /Watchdog/WD_FAULT
- U2 pad 1: +3.3V -> GND
- U2 pad 2: Net-(U2-CWD) -> /SW_CHRG_2
- U2 pad 3: /Watchdog/SET0 -> +3.3V
- U2 pad 4: Net-(Q9-D) -> unconnected-(U2-Pad4)_1
- U2 pad 5: GND -> unconnected-(U2-Pad5)
- U3 pad 1: +5V -> GND
- U3 pad 2: unconnected-(U3-Pad2) -> /SW_CHRG_3
- U3 pad 3: Net-(J3-Pin_1) -> +3.3V
- U3 pad 4: Net-(U3-Pad4) -> unconnected-(U3-Pad4)_1
- U3 pad 5: Net-(U3-Pad4) -> unconnected-(U3-Pad5)_1
- U4 pad 1: GND -> +5V
- U4 pad 2: Net-(Q10-G) -> unconnected-(U4-Pad2)
- U4 pad 3: +3.3V -> Net-(J8-Pin_1)
Routing:
- added copper zone on B.Cu, net +5V
- added copper zone on F.Cu, net +5V
Other:
- board size 135 x 56 mm -> 128.5 x 56 mm
- board text added: "5V BUCK"

Commit message: cs: finalized PI HAT
Parts:
- added D2: D_Schottky, Diode_SMD:D_SOD-323, F.Cu at (183.5, 144.1)
- added D3: WD_LED_EN, LED_SMD:LED_0805_2012Metric, F.Cu at (231.6, 161.0)
- added D4: WDO, LED_SMD:LED_0805_2012Metric, F.Cu at (231.6, 165.8)
- added D5: Heartbeat, LED_SMD:LED_0805_2012Metric, F.Cu at (231.6, 163.4)
- added JP1: force enable, Jumper:SolderJumper-2_P1.3mm_Open_RoundedPad1.0x1.5mm, F.Cu at (184.5, 160.6)
- added R10: 200, Resistor_SMD:R_0603_1608Metric, F.Cu at (213.0, 157.7)
- added R11: 200, Resistor_SMD:R_0603_1608Metric, F.Cu at (213.0, 156.1)
- added R3: 200, Resistor_SMD:R_0603_1608Metric, F.Cu at (184.4, 146.7)
- added R4: 10k, Resistor_SMD:R_0805_2012Metric_Pad1.20x1.40mm_HandSolder, F.Cu at (195.8, 149.2)
- added R5: 10k, Resistor_SMD:R_0805_2012Metric, F.Cu at (204.3, 149.5)
- added R6: 10k, Resistor_SMD:R_0805_2012Metric, F.Cu at (202.8, 155.8)
- added R8: 200, Resistor_SMD:R_0603_1608Metric, F.Cu at (204.3, 151.4)
- added R9: 200, Resistor_SMD:R_0603_1608Metric, F.Cu at (190.9, 154.2)
- added TP1: SET0, TestPoint:TestPoint_Pad_D1.0mm, B.Cu at (190.3, 149.7)
- added TP2: WD_EN, TestPoint:TestPoint_Pad_D1.0mm, B.Cu at (190.3, 156.6)
- added TP3: ~{WDO}, TestPoint:TestPoint_Pad_D1.0mm, B.Cu at (209.0, 150.4)
- added kibuzzard-6AD528DF: G***, kibuzzard-6AD528DF, F.Cu at (196.3, 160.6)
- added kibuzzard-6AD530C8: G***, kibuzzard-6AD530C8, F.Cu at (226.0, 161.0)
- added kibuzzard-6AD530EA: G***, kibuzzard-6AD530EA, F.Cu at (223.6, 163.4)
- added kibuzzard-6AD5310E: G***, kibuzzard-6AD5310E, F.Cu at (223.6, 165.8)
- added kibuzzard-6AD537E7: G***, kibuzzard-6AD537E7, F.Cu at (226.1, 158.4)
- added kibuzzard-6AD53C20: G***, kibuzzard-6AD53C20, F.Cu at (172.0, 168.9)
- added kibuzzard-6AD53C20: G***, kibuzzard-6AD53C20, B.Cu at (171.9, 162.9)
- added kibuzzard-6AD53C20: G***, kibuzzard-6AD53C20, B.Cu at (268.3, 161.8)
- added kibuzzard-6AD53C3D: G***, kibuzzard-6AD53C3D, F.Cu at (197.0, 168.9)
- added kibuzzard-6AD53C43: G***, kibuzzard-6AD53C43, F.Cu at (229.5, 168.9)
- added kibuzzard-6AD53C84: G***, kibuzzard-6AD53C84, F.Cu at (268.3, 168.9)
- added kibuzzard-6AD53CF1: G***, kibuzzard-6AD53CF1, F.Cu at (272.5, 137.9)
- added kibuzzard-6AD53D49: G***, kibuzzard-6AD53D49, F.Cu at (260.0, 138.0)
- added kibuzzard-6AD53DF3: G***, kibuzzard-6AD53DF3, F.Cu at (223.2, 134.6)
- added kibuzzard-6AD53E3A: G***, kibuzzard-6AD53E3A, F.Cu at (235.7, 134.6)
- added kibuzzard-6AD53E40: G***, kibuzzard-6AD53E40, F.Cu at (248.2, 134.6)
- added kibuzzard-6AD5403C: G***, kibuzzard-6AD5403C, F.Cu at (218.3, 149.9)
- added kibuzzard-6AD54089: G***, kibuzzard-6AD54089, F.Cu at (232.8, 152.4)
- added kibuzzard-6AD540AE: G***, kibuzzard-6AD540AE, F.Cu at (232.8, 147.4)
- added kibuzzard-6AD541D1: G***, kibuzzard-6AD541D1, F.Cu at (242.5, 177.0)
- added kibuzzard-6AD543B1: G***, kibuzzard-6AD543B1, B.Cu at (197.0, 162.9)
- added kibuzzard-6AD543B7: G***, kibuzzard-6AD543B7, B.Cu at (229.5, 162.9)
- H1: footprint MountingHole:MountingHole_2.2mm_M2_DIN965 -> MountingHole:MountingHole_2.2mm_M2_DIN965_Pad
- H2: footprint MountingHole:MountingHole_2.5mm -> MountingHole:MountingHole_2.5mm_Pad
- J1, J2, J3, J8: footprint TerminalBlock_Phoenix:TerminalBlock_Phoenix_PT-1,5-2-3.5-H_1x02_P3.50mm_Horizontal -> TerminalBlock_Phoenix:TerminalBlock_Phoenix_PT-1,5-2-5.0-H_1x02_P5.00mm_Horizontal
- J4: value RFID1 -> RFID0
- J5: value RFID2 -> RFID1
- J6: value RFID3 -> RFID2
- moved Q5 100.2 mm to (181.6, 154.2), turned to 180 degrees
- moved Q3 97.0 mm to (177.5, 151.0), turned to -90 degrees
- moved Q8 92.7 mm to (238.8, 164.8)
- moved Q7 92.4 mm to (205.9, 154.6), turned to -90 degrees
- moved Q4 91.8 mm to (186.1, 154.2)
- moved Q6 89.9 mm to (199.4, 155.8), turned to 180 degrees
- moved Q1 89.4 mm to (186.1, 149.5)
- moved Q2 87.4 mm to (181.6, 149.5), turned to 180 degrees
- moved U6 86.9 mm to (176.5, 147.0), turned to -90 degrees
- moved C2 86.0 mm to (173.8, 146.9), turned to -90 degrees
- moved C4 80.8 mm to (193.7, 153.8), turned to -90 degrees
- moved C5 71.4 mm to (199.3, 148.3)
- moved C3 63.1 mm to (195.8, 153.1), turned to -90 degrees
- moved U7 62.5 mm to (200.0, 151.4)
- moved J2 12.3 mm to (275.0, 132.8)
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Connections:
- net /Raspi5/GPIO10/SPI0.MOSI renamed /Raspi5/D_MOSI
- net /Raspi5/GPIO11/SPI0.SCLK renamed /Raspi5/D_CLK
- net /Raspi5/GPIO24 renamed /Raspi5/D_LCD_RS
- net /Raspi5/GPIO25 renamed /Raspi5/D_RST
- net /Raspi5/GPIO7/SPI0.CE1 renamed /Raspi5/D_TP_CS
- net /Raspi5/GPIO8/SPI0.CE0 renamed /Raspi5/D_LCD_CS
- net /Raspi5/GPIO9/SPI0.MISO renamed /Raspi5/D_TP_SO
- J4 pad 2: /CE1 -> /CE0
- J5 pad 2: /CE2 -> /CE1
- J6 pad 2: /CE3 -> /CE2
- J9 pad 10: /Raspi5/GPIO15/WD_EN -> /Raspi5/GPIO2/MPPT
- J9 pad 11: unconnected-(J9-Pin_11-Pad11) -> /Raspi5/D_TP_IRQ
- J9 pad 12: /CE1 -> /Raspi5/GPIO18/GPIO_WD_EN
- J9 pad 13: /SW_CHRG_3 -> /Raspi5/GPIO14/GPIO_WD
- J9 pad 15: /SW_CHRG_2 -> /B_GREEN
- J9 pad 16: /SW_CHRG_1 -> /S_GREEN
- J9 pad 27: /B_RED -> /S_YELLOW
- J9 pad 28: /S_YELLOW -> /B_YELLOW
- J9 pad 29: /CE2 -> /B_RED
- J9 pad 3: /Raspi5/GPIO2/MPPT -> /SW_CHRG_1
- J9 pad 31: /B_YELLOW -> /S_RED
- J9 pad 33: /S_GREEN -> /CE1
- J9 pad 36: /CE3 -> /CE2
- J9 pad 37: /B_GREEN -> /CE0
- J9 pad 5: /Raspi5/GPIO3/PS -> /SW_CHRG_2
- J9 pad 7: /S_RED -> /SW_CHRG_3
- J9 pad 8: /Raspi5/GPIO14/GPIO_WD -> /Raspi5/GPIO3/PS
- Q4 pad 3: Net-(D2-K) -> Net-(Q1-G)
- Q5 pad 3: Net-(D2-K) -> Net-(Q1-G)
- Q7 pad 1: Net-(Q7-G) -> Net-(D4-K)
- Q8 pad 1: Net-(Q8-G) -> Net-(D4-K)
Routing:
- net +3.3V: track 0.00 -> 328.0 mm, vias 0 -> 6
- net /RST: track 0.00 -> 132.4 mm, vias 0 -> 2
- net /B_YELLOW: track 0.00 -> 126.1 mm
- net /MISO: track 0.00 -> 124.0 mm, vias 0 -> 2
- net /MOSI: track 0.00 -> 123.8 mm, vias 0 -> 2
- net /S_YELLOW: track 0.00 -> 122.3 mm
- net /B_RED: track 0.00 -> 122.1 mm
- net /S_RED: track 0.00 -> 121.8 mm
- net /CLK: track 0.00 -> 119.4 mm, vias 0 -> 2
- net /S_GREEN: track 0.00 -> 117.5 mm
- net /B_GREEN: track 0.00 -> 115.2 mm
- net /CE2: track 0.00 -> 92.1 mm
- net /Raspi5/GPIO2/MPPT: track 0.00 -> 81.2 mm
- net +5V: track 0.00 -> 75.6 mm
- net /Raspi5/GPIO3/PS: track 0.00 -> 65.3 mm
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- added copper zone on B.Cu, net +3.3V
- added copper zone on F.Cu, net +3.3V
- added copper zone on F.Cu, net /Watchdog/SET0
- added copper zone on F.Cu, net Net-(U4-Pad5)
Other:
- board text added: "+3.3V"
- board text added: "B_{AMBER}"
- board text added: "B_{GREEN}"
- board text added: "B_{RED}"
- board text added: "CLK"
- board text added: "CS"
- board text added: "EN_{WD}"
- board text added: "GND"
- board text added: "MISO"
- board text added: "MOSI"
- board text added: "OFF"
- board text added: "ON"
- board text added: "RST"
- board text added: "SET0"
- board text added: "S_{AMBER}"
- board text added: "S_{GREEN}"
- board text added: "S_{RED}"
- board text added: "~{WDO}"
