File: charging_station/KiCad/PIHAT/PIHAT.kicad_sch (KiCad schematic)
At the start: 13 parts, among them J2 5v(Vin), J3 WD_F, J4 Raspberry Control Signals, J5 RFID1, J6 RFID2, J7 MPPT, J8 PS, J9 RFID3, SW2 Sw_1, SW6 Sw_1, SW7 Sw_1, U3 IM03GR

Commit message: cd: hat: finalized schematic + rough layout
Parts:
- removed J2: 5v(Vin), TerminalBlock_Phoenix:TerminalBlock_Phoenix_PT-1,5-2-3.5-H_1x02_P3.50mm_Horizontal, symbol Connector:Screw_Terminal_01x02
- removed SW2, SW6, SW7: Sw_1, Button_Switch_SMD:SW_SPDT_CK_JS102011SAQN, symbol Switch:SW_SPDT_MSM
- added H1: MountingHole, MountingHole:MountingHole_2.2mm_M2_DIN965, symbol Mechanical:MountingHole
- added H2: MountingHole, MountingHole:MountingHole_2.5mm, symbol Mechanical:MountingHole
- added J1: 5v(Vin), TerminalBlock_Phoenix:TerminalBlock_Phoenix_PT-1,5-2-3.5-H_1x02_P3.50mm_Horizontal, symbol Connector:Screw_Terminal_01x02
- added U1, U2, U3: MSK12C02G25-B, external_ECAD:SW-SMD_MSK12C02G25-B, symbol external_ECAD:MSK12C02G25-B
- renumbered J7 to J2, J8 to J3, J5 to J4, J6 to J5, J9 to J6, J4 to J7, J3 to J8, U3 to U4
Connections:
- net +3.3V: now also U1.3, U2.3, U3.3
- net +5V: now also J1.1 (Pin_1)
- net GND: now also J1.2 (Pin_2), U1.1, U2.1, U3.1
- net SW_CHRG_1: now also U1.2
- net SW_CHRG_2: now also U2.2
- net SW_CHRG_3: now also U3.2
- net at U4.4: now also J8.2 (Pin_2); no longer U4.5
- net at U4.6: now also U4.5; no longer J8.2 (Pin_2)
- no-connect marks 2 -> 8
Other:
- moved on the sheet: J8

Commit message: cs: finalized PI HAT
Parts:
- D1: LCSC C95872 -> (none); LCSC Part (none) -> C95872
- H1: footprint MountingHole:MountingHole_2.2mm_M2_DIN965 -> MountingHole:MountingHole_2.2mm_M2_DIN965_Pad
- H2: footprint MountingHole:MountingHole_2.5mm -> MountingHole:MountingHole_2.5mm_Pad
- J1, J2, J3, J8: footprint TerminalBlock_Phoenix:TerminalBlock_Phoenix_PT-1,5-2-3.5-H_1x02_P3.50mm_Horizontal -> TerminalBlock_Phoenix:TerminalBlock_Phoenix_PT-1,5-2-5.0-H_1x02_P5.00mm_Horizontal; LCSC Part (none) -> C5188434; MPN (none) -> MX126-5.0-02P-GN01-Cu-S-A
- J4: value RFID1 -> RFID0
- J5: value RFID2 -> RFID1
- J6: value RFID3 -> RFID2
Connections:
- net CE3 is gone; now on net CE2: J6.2 (Pin_2)
- net CE1: now also J5.2 (Pin_2); no longer J4.2 (Pin_2)
- net CE2: no longer J5.2 (Pin_2)
- net at U4.4: now also U4.5; no longer J8.2 (Pin_2)
- net at U4.6: now also J8.2 (Pin_2); no longer U4.5
- new net CE0: J4.2 (Pin_2)
- no-connect marks 8 -> 2
Other:
- sheet Raspi5 ports: added GPIO0/Y_B, GPIO13/R_B, GPIO18/GPIO_WD_EN, GPIO1/G_S, GPIO26/R_S, GPIO4/G_B, GPIO6/Y_S, SW_BUCK_10, SW_BUCK_11, SW_BUCK_12; removed GPIO0/R_MO, GPIO13/G_ST, GPIO15/WD_EN, GPIO1/Y_ST, GPIO26/G_MO, GPIO4/R_ST, GPIO6/Y_MO, SW_CHRG_1, SW_CHRG_2, SW_CHRG_3
- moved on the sheet: J8

Commit message: cs: finalized KiCad files
Changed lines of the file:
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@@
 		)
 		(instances
-			(project "PIHAT-rounded"
+			(project "PIHAT"
 				(path "/e63e39d7-6ac0-4ffd-8aa3-1841a4541b55"
 					(reference "J1")
@@
 		)
 		(instances
-			(project "PIHAT-rounded"
+			(project "PIHAT"
 				(path "/e63e39d7-6ac0-4ffd-8aa3-1841a4541b55"
 					(reference "#FLG01")
@@
 		)
 		(instances
-			(project "PIHAT-rounded"
+			(project "PIHAT"
 				(path "/e63e39d7-6ac0-4ffd-8aa3-1841a4541b55"
 					(reference "#PWR013")
@@
 		)
 		(instances
-			(project "PIHAT-rounded"
+			(project "PIHAT"
 				(path "/e63e39d7-6ac0-4ffd-8aa3-1841a4541b55"
 					(reference "U4")
@@
 		)
 		(instances
-			(project "PIHAT-rounded"
+			(project "PIHAT"
 				(path "/e63e39d7-6ac0-4ffd-8aa3-1841a4541b55"
 					(reference "#PWR08")
@@
 		)
 		(instances
-			(project "PIHAT-rounded"
+			(project "PIHAT"
 				(path "/e63e39d7-6ac0-4ffd-8aa3-1841a4541b55"
 					(reference "#PWR011")
@@
 		(dnp no)
 		(property "Reference" "U2"
-			(at 50.8 93.98 0)
+			(at 37.846 78.994 90)
 			(show_name no)
 			(do_not_autoplace no)
@@
 		)
 		(property "Value" "MSK12C02G25-B"
-			(at 30.48 93.98 0)
+			(at 38.1 80.772 90)
 			(show_name no)
 			(do_not_autoplace no)
@@
 		)
 		(instances
-			(project "PIHAT-rounded"
+			(project "PIHAT"
 				(path "/e63e39d7-6ac0-4ffd-8aa3-1841a4541b55"
 					(reference "U2")
@@
 		)
 		(instances
-			(project "PIHAT-rounded"
+			(project "PIHAT"
 				(path "/e63e39d7-6ac0-4ffd-8aa3-1841a4541b55"
 					(reference "#PWR07")
@@
 		)
 		(instances
-			(project "PIHAT-rounded"
+			(project "PIHAT"
 				(path "/e63e39d7-6ac0-4ffd-8aa3-1841a4541b55"
 					(reference "#PWR015")
@@
 		)
 		(instances
-			(project "PIHAT-rounded"
+			(project "PIHAT"
 				(path "/e63e39d7-6ac0-4ffd-8aa3-1841a4541b55"
 					(reference "#PWR04")
@@
 		)
 		(instances
-			(project "PIHAT-rounded"
+			(project "PIHAT"
 				(path "/e63e39d7-6ac0-4ffd-8aa3-1841a4541b55"
 					(reference "H1")
@@
 		(dnp no)
 		(property "Reference" "U1"
-			(at 50.8 60.96 0)
+			(at 38.1 45.212 90)
 			(show_name no)
 			(do_not_autoplace no)
@@
 		)
 		(property "Value" "MSK12C02G25-B"
-			(at 30.48 60.96 0)
+			(at 38.354 47.244 90)
 			(show_name no)
 			(do_not_autoplace no)
@@
 		)
 		(instances
-			(project "PIHAT-rounded"
+			(project "PIHAT"
 				(path "/e63e39d7-6ac0-4ffd-8aa3-1841a4541b55"
 					(reference "U1")
@@
 		)
 		(instances
-			(project "PIHAT-rounded"
+			(project "PIHAT"
 				(path "/e63e39d7-6ac0-4ffd-8aa3-1841a4541b55"
 					(reference "#PWR017")
@@
 		)
 		(instances
-			(project "PIHAT-rounded"
+			(project "PIHAT"
 				(path "/e63e39d7-6ac0-4ffd-8aa3-1841a4541b55"
 					(reference "J7")
@@
 		)
 		(instances
-			(project "PIHAT-rounded"
+			(project "PIHAT"
 				(path "/e63e39d7-6ac0-4ffd-8aa3-1841a4541b55"
 					(reference "J6")
@@
 		)
 		(instances
-			(project "PIHAT-rounded"
+			(project "PIHAT"
 				(path "/e63e39d7-6ac0-4ffd-8aa3-1841a4541b55"
 					(reference "J3")
@@
 		(dnp no)
 		(property "Reference" "U3"
-			(at 50.8 127 0)
+			(at 37.846 111.506 90)
 			(show_name no)
 			(do_not_autoplace no)
@@
 		)
 		(property "Value" "MSK12C02G25-B"
-			(at 30.48 127 0)
+			(at 38.1 113.538 90)
 			(show_name no)
 			(do_not_autoplace no)
@@
 		)
 		(instances
-			(project "PIHAT-rounded"
+			(project "PIHAT"
 				(path "/e63e39d7-6ac0-4ffd-8aa3-1841a4541b55"
 					(reference "U3")
@@
 		)
 		(instances
-			(project "PIHAT-rounded"
+			(project "PIHAT"
 				(path "/e63e39d7-6ac0-4ffd-8aa3-1841a4541b55"
 					(reference "#PWR014")
@@
 		)
 		(instances
-			(project "PIHAT-rounded"
+			(project "PIHAT"
 				(path "/e63e39d7-6ac0-4ffd-8aa3-1841a4541b55"
 					(reference "J4")
@@
 		)
 		(instances
-			(project "PIHAT-rounded"
+			(project "PIHAT"
 				(path "/e63e39d7-6ac0-4ffd-8aa3-1841a4541b55"
 					(reference "#FLG02")
@@
 		)
 		(instances
-			(project "PIHAT-rounded"
+			(project "PIHAT"
 				(path "/e63e39d7-6ac0-4ffd-8aa3-1841a4541b55"
 					(reference "#PWR09")
@@
 		)
 		(instances
-			(project "PIHAT-rounded"
+			(project "PIHAT"
 				(path "/e63e39d7-6ac0-4ffd-8aa3-1841a4541b55"
 					(reference "#PWR016")
@@
 		)
 		(instances
-			(project "PIHAT-rounded"
+			(project "PIHAT"
 				(path "/e63e39d7-6ac0-4ffd-8aa3-1841a4541b55"
 					(reference "#PWR012")
@@
 		)
 		(instances
-			(project "PIHAT-rounded"
+			(project "PIHAT"
 				(path "/e63e39d7-6ac0-4ffd-8aa3-1841a4541b55"
 					(reference "D1")
@@
 		)
 		(instances
-			(project "PIHAT-rounded"
+			(project "PIHAT"
 				(path "/e63e39d7-6ac0-4ffd-8aa3-1841a4541b55"
 					(reference "#PWR01")
@@
 		)
 		(instances
-			(project "PIHAT-rounded"
+			(project "PIHAT"
 				(path "/e63e39d7-6ac0-4ffd-8aa3-1841a4541b55"
 					(reference "#PWR03")
@@
 		)
 		(instances
-			(project "PIHAT-rounded"
+			(project "PIHAT"
 				(path "/e63e39d7-6ac0-4ffd-8aa3-1841a4541b55"
 					(reference "#PWR05")
@@
 		)
 		(instances
-			(project "PIHAT-rounded"
+			(project "PIHAT"
 				(path "/e63e39d7-6ac0-4ffd-8aa3-1841a4541b55"
 					(reference "J2")
@@
 		)
 		(instances
-			(project "PIHAT-rounded"
+			(project "PIHAT"
 				(path "/e63e39d7-6ac0-4ffd-8aa3-1841a4541b55"
 					(reference "#PWR02")
@@
 		)
 		(instances
-			(project "PIHAT-rounded"
+			(project "PIHAT"
 				(path "/e63e39d7-6ac0-4ffd-8aa3-1841a4541b55"
 					(reference "J5")
@@
 		)
 		(instances
-			(project "PIHAT-rounded"
+			(project "PIHAT"
 				(path "/e63e39d7-6ac0-4ffd-8aa3-1841a4541b55"
 					(reference "#PWR018")
@@
 		)
 		(instances
-			(project "PIHAT-rounded"
+			(project "PIHAT"
 				(path "/e63e39d7-6ac0-4ffd-8aa3-1841a4541b55"
 					(reference "J8")
@@
 		)
 		(instances
-			(project "PIHAT-rounded"
+			(project "PIHAT"
 				(path "/e63e39d7-6ac0-4ffd-8aa3-1841a4541b55"
 					(reference "H2")
@@
 		)
 		(instances
-			(project "PIHAT-rounded"
+			(project "PIHAT"
 				(path "/e63e39d7-6ac0-4ffd-8aa3-1841a4541b55"
 					(reference "#PWR010")
@@
 		)
 		(instances
-			(project "PIHAT-rounded"
+			(project "PIHAT"
 				(path "/e63e39d7-6ac0-4ffd-8aa3-1841a4541b55"
 					(reference "#PWR06")
@@
 		)
 		(instances
-			(project "PIHAT-rounded"
+			(project "PIHAT"
 				(path "/e63e39d7-6ac0-4ffd-8aa3-1841a4541b55"
 					(page "4")
@@
 		)
 		(instances
-			(project "PIHAT-rounded"
+			(project "PIHAT"
 				(path "/e63e39d7-6ac0-4ffd-8aa3-1841a4541b55"
 					(page "2")
