File: charging_station/KiCad/PIHAT/raspi5.kicad_sch (KiCad schematic)
At the start: 6 parts, among them J1 GPIO, U1 CAT24C256

Commit message: cd: hat: finalized schematic + rough layout
Parts:
- renumbered J1 to J9, U1 to U5
Changed lines of the file:
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@@
 		(dnp no)
 		(fields_autoplaced yes)
-		(property "Reference" "#PWR08"
+		(property "Reference" "#PWR022"
 			(at 134.62 68.58 0)
 			(hide yes)
@@
 			(project "PIHAT"
 				(path "/e63e39d7-6ac0-4ffd-8aa3-1841a4541b55/8b73852e-04bf-4357-a410-53a0a560e029"
-					(reference "#PWR08")
+					(reference "#PWR022")
 					(unit 1)
 				)
@@
 		(in_pos_files no)
 		(dnp yes)
-		(property "Reference" "#PWR0102"
+		(property "Reference" "#PWR019"
 			(at 87.63 195.58 0)
 			(hide yes)
@@
 			(project "PIHAT"
 				(path "/e63e39d7-6ac0-4ffd-8aa3-1841a4541b55/8b73852e-04bf-4357-a410-53a0a560e029"
-					(reference "#PWR0102")
+					(reference "#PWR019")
 					(unit 1)
 				)
@@
 		(in_pos_files yes)
 		(dnp no)
-		(property "Reference" "J1"
+		(property "Reference" "J9"
 			(at 146.05 65.6398 0)
 			(show_name no)
@@
 			(project "PIHAT"
 				(path "/e63e39d7-6ac0-4ffd-8aa3-1841a4541b55/8b73852e-04bf-4357-a410-53a0a560e029"
-					(reference "J1")
+					(reference "J9")
 					(unit 1)
 				)
@@
 		(in_pos_files yes)
 		(dnp no)
-		(property "Reference" "#PWR03"
+		(property "Reference" "#PWR023"
 			(at 137.16 129.54 0)
 			(hide yes)
@@
 			(project "PIHAT"
 				(path "/e63e39d7-6ac0-4ffd-8aa3-1841a4541b55/8b73852e-04bf-4357-a410-53a0a560e029"
-					(reference "#PWR03")
+					(reference "#PWR023")
 					(unit 1)
 				)
@@
 		(in_pos_files no)
 		(dnp yes)
-		(property "Reference" "#PWR0103"
+		(property "Reference" "#PWR021"
 			(at 104.14 179.07 0)
 			(hide yes)
@@
 			(project "PIHAT"
 				(path "/e63e39d7-6ac0-4ffd-8aa3-1841a4541b55/8b73852e-04bf-4357-a410-53a0a560e029"
-					(reference "#PWR0103")
+					(reference "#PWR021")
 					(unit 1)
 				)
@@
 		(in_pos_files yes)
 		(dnp no)
-		(property "Reference" "#PWR02"
+		(property "Reference" "#PWR025"
 			(at 154.94 129.54 0)
 			(hide yes)
@@
 			(project "PIHAT"
 				(path "/e63e39d7-6ac0-4ffd-8aa3-1841a4541b55/8b73852e-04bf-4357-a410-53a0a560e029"
-					(reference "#PWR02")
+					(reference "#PWR025")
 					(unit 1)
 				)
@@
 		(dnp no)
 		(fields_autoplaced yes)
-		(property "Reference" "#PWR09"
+		(property "Reference" "#PWR024"
 			(at 154.94 68.58 0)
 			(hide yes)
@@
 			(project "PIHAT"
 				(path "/e63e39d7-6ac0-4ffd-8aa3-1841a4541b55/8b73852e-04bf-4357-a410-53a0a560e029"
-					(reference "#PWR09")
+					(reference "#PWR024")
 					(unit 1)
 				)
@@
 		(in_pos_files no)
 		(dnp yes)
-		(property "Reference" "U1"
+		(property "Reference" "U5"
 			(at 81.28 169.5258 0)
 			(show_name no)
@@
 			(project "PIHAT"
 				(path "/e63e39d7-6ac0-4ffd-8aa3-1841a4541b55/8b73852e-04bf-4357-a410-53a0a560e029"
-					(reference "U1")
+					(reference "U5")
 					(unit 1)
 				)
@@
 		(in_pos_files no)
 		(dnp yes)
-		(property "Reference" "#PWR0101"
+		(property "Reference" "#PWR020"
 			(at 107.95 165.1 0)
 			(hide yes)
@@
 			(project "PIHAT"
 				(path "/e63e39d7-6ac0-4ffd-8aa3-1841a4541b55/8b73852e-04bf-4357-a410-53a0a560e029"
-					(reference "#PWR0101")
-					(unit 1)
-				)
+					(reference "#PWR020")
+					(unit 1)
+				)

Commit message: cs: finalized PI HAT
Parts:
- removed C1: 100n, symbol Device:C_Small
- removed JP1: ID_WP, symbol Jumper:SolderJumper_2_Open
- removed R1, R2: 3.9k, symbol Device:R_Small
- removed U5: CAT24C256, symbol Memory_EEPROM:CAT24C256
- J9: LCSC (none) -> C6235776; MPN (none) -> SSQ-120-03-T-D
Connections:
- net GPIO13/G_ST is gone; now on net GPIO5/CE1: J9.33 (Pin_33)
- net GPIO15/WD_EN is gone; now on net GPIO2/MPPT: J9.10 (Pin_10)
- net GPIO26/G_MO is gone; now on net GPIO18/CE0: J9.37 (Pin_37)
- net SW_CHRG_3 is gone; now on net GPIO14/GPIO_WD: J9.13 (Pin_13)
- net GPIO14/GPIO_WD: no longer J9.8 (Pin_8)
- net GPIO18/CE0: no longer J9.12 (Pin_12)
- net GPIO2/MPPT: no longer J9.3 (Pin_3)
- net GPIO3/PS: now also J9.8 (Pin_8); no longer J9.5 (Pin_5)
- net GPIO5/CE1: no longer J9.29 (Pin_29)
- net D_TP_IRQ: now reaches J9.11 (Pin_11)
- net GPIO0/R_MO renamed GPIO6/Y_S
- net GPIO10/SPI0.MOSI renamed D_MOSI
- net GPIO11/SPI0.SCLK renamed D_CLK
- net GPIO1/Y_ST renamed GPIO0/Y_B
- net GPIO24 renamed D_LCD_RS
- net GPIO25 renamed D_RST
- net GPIO4/R_ST renamed SW_BUCK_12
- net GPIO6/Y_MO renamed GPIO26/R_S
- net GPIO7/SPI0.CE1 renamed D_TP_CS
- net GPIO8/SPI0.CE0 renamed D_LCD_CS
- net GPIO9/SPI0.MISO renamed D_MISO
- net SW_CHRG_1 renamed GPIO1/G_S
- net SW_CHRG_2 renamed GPIO4/G_B
- new net GPIO13/R_B: J9.29 (Pin_29)
- new net GPIO18/GPIO_WD_EN: J9.12 (Pin_12)
- new net SW_BUCK_10: J9.3 (Pin_3)
- new net SW_BUCK_11: J9.5 (Pin_5)
- no-connect marks 4 -> 8
Other:
- note added: "D_* annotates Display hat pins"
- note removed: "ID_SD and ID_SC PINS: These pins are reserved for HAT ID EEPROM. At boot time this I2C interface will be interrogated to look for an EEPROM that identifes the attached board and allows automagic setup of the GPIOs (and optionally, Linux drivers). Bridging JP1 enables write protection. DO NOT USE these pins for anything other than attaching an I2C ID EEPROM. Leave unconnected if ID EEPROM not requ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"
