File: charging_station/KiCad/PIHAT/watchdog.kicad_sch (KiCad schematic)
At the start: 21 parts, among them Q1 AO3400A, Q10 AO3401A, Q4 AO3401A, Q5 AO3400A, Q6 AO3401A, Q7 AO3400A, Q8 AO3401A, Q9 AO3400A, U2 TPS3430WDRC, U4 TLV809EA29DBZR

Commit message: cd: hat: finalized schematic + rough layout
Parts:
- renumbered C4 to C2, C2 to C3, C5 to C4, C3 to C5, Q4 to Q1, Q5 to Q2, Q10 to Q3, Q6 to Q4, Q7 to Q5, Q9 to Q6, Q8 to Q7, Q1 to Q8, R10 to R3, R9 to R4, R11 to R5, R12 to R6, R4 to R8, U4 to U6, U2 to U7

Commit message: cs: finalized PI HAT
Parts:
- removed R7: 100, symbol Device:R_Small
- added D3: WD_LED_EN, LED_SMD:LED_0805_2012Metric, symbol Device:LED
- added D4: WDO, LED_SMD:LED_0805_2012Metric, symbol Device:LED
- added D5: Heartbeat, LED_SMD:LED_0805_2012Metric, symbol Device:LED
- added JP1: force enable, Jumper:SolderJumper-2_P1.3mm_Open_RoundedPad1.0x1.5mm, symbol Jumper:SolderJumper_2_Open
- added R10, R11, R9: 200, Resistor_SMD:R_0603_1608Metric, symbol Device:R_Small
- added TP1: SET0, TestPoint:TestPoint_Pad_D1.0mm, symbol Connector:TestPoint
- added TP2: WD_EN, TestPoint:TestPoint_Pad_D1.0mm, symbol Connector:TestPoint
- added TP3: ~{WDO}, TestPoint:TestPoint_Pad_D1.0mm, symbol Connector:TestPoint
- C2, C5: LCSC C14663 -> (none); LCSC Part (none) -> C14663
- D2: footprint (none) -> Diode_SMD:D_SOD-323
- Q1, Q3, Q4, Q7: LCSC C15127 -> (none); LCSC Part (none) -> C15127
- Q2, Q5, Q6, Q8: LCSC C20917 -> (none); LCSC Part (none) -> C15127
- R3, R8: value 100 -> 200; footprint (none) -> Resistor_SMD:R_0603_1608Metric
- R4: footprint (none) -> Resistor_SMD:R_0805_2012Metric_Pad1.20x1.40mm_HandSolder
- R5, R6: footprint (none) -> Resistor_SMD:R_0805_2012Metric
Connections:
- net +3.3V: now also D4.2 (A)
- net GND: now also D3.1 (K), D5.1 (K), JP1.2 (B)
- net GPIO_WD: now also R10.2, R11.2
- net SET0: now also JP1.1 (A), TP1.1
- net at Q7.1 (G): now also Q8.1 (G), R5.2, R8.2, D4.1 (K), TP3.1
- net at R8.1, U7.8 (~{WDO}): no longer R5.2
- net at Q1.1 (G), Q2.1 (G), R3.2: now also Q4.3 (D), Q5.3 (D), R9.1, TP2.1
- net at D2.1 (K), R3.1: no longer Q4.3 (D), Q5.3 (D)
- new net: D5.2 (A), R10.1, R11.1
- new net: D3.2 (A), R9.2
Other:
- note added: "100 Ohm"
- note added: "LED Red => 140 < R < 300 @ 5mA"
- note added: "LED Yellow => 180 < R < 260 @ 5mA"
- moved on the sheet: D2, R3
