File: charging_station/KiCad/SLCU/GPIO_MUX.kicad_sch (KiCad schematic)
At the start: 31 parts, among them Q11 2N7002, Q12 2N7002, Q13 2N7002, Q14 2N7002, Q15 2N7002, Q16 2N7002, Q17 2N7002

Commit message: cs: corrected wrong mosfets on SLCU
Parts:
- Q15: value 2N7002 -> 2SK1958-VB; LCSC Part (none) -> C20755445; MPN (none) -> 2SK1958-VB
Other:
- note added: "max PD_{12V} = 12V * ((12V-2V)/1500ohm + 12V/1000ohm) = @{format(12 * ((12-2)/1500 + 12/1000), 3)}W max PD_{10V} = 10V * ((10V-2V)/1500ohm + 10V/1000ohm) = @{format(10 * ((10-2)/1500 + 10/1000), 3)}W"
- note added: "max PD_{12V} = 12V * (7*(12V-2V)/1500ohm) + 6*12V/1000ohm) = @{format(12 * (7*(12-2)/1500 + 6*12/1000), 3)} W max PD_{10V} = 10V * (7*(10V-2V)/1500ohm) + 6*10V/1000ohm) = @{format(10 * (7*(10-2)/1500 + 6*10/1000), 3)} W"
Changed lines of the file:
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@@
 		(title "SLCU (Stack Light Control Unit)")
 		(date "2026-10-10")
-		(rev "3.0")
+		(rev "3.1")
 		(company "JMU Würzburg")
 		(comment 1 "Nico Schubert")
@@
 		)
 	)
+	(text "max PD_{12V} = 12V * (7*(12V-2V)/1500ohm) + 6*12V/1000ohm) = @{format(12 * (7*(12-2)/1500 + 6*12/1000), 3)} W\nmax PD_{10V} = 10V * (7*(10V-2V)/1500ohm) + 6*10V/1000ohm) = @{format(10 * (7*(10-2)/1500 + 6*10/1000), 3)} W\n"
+		(exclude_from_sim no)
+		(at 108.204 34.798 0)
+		(effects
+			(font
+				(size 1.27 1.27)
+			)
+			(justify left bottom)
+		)
+	)
 	(text "Signal Translator: Enable Gate"
 		(exclude_from_sim no)
@@
 		)
 	)
+	(text "max PD_{12V} = 12V * ((12V-2V)/1500ohm + 12V/1000ohm) = @{format(12 * ((12-2)/1500 + 12/1000), 3)}W\nmax PD_{10V} = 10V * ((10V-2V)/1500ohm + 10V/1000ohm) = @{format(10 * ((10-2)/1500 + 10/1000), 3)}W"
+		(exclude_from_sim no)
+		(at 39.37 78.994 0)
+		(effects
+			(font
+				(size 1.27 1.27)
+			)
+			(justify left bottom)
+		)
+	)
 	(text "Singal Translator: RED"
 		(exclude_from_sim no)
@@
 			)
 		)
-		(property "Value" "2N7002"
+		(property "Value" "2SK1958-VB"
 			(at 146.05 44.704 90)
 			(show_name no)
@@
 			(at 146.05 50.8 0)
 			(hide yes)
+			(show_name no)
+			(do_not_autoplace no)
+			(effects
+				(font
+					(size 1.27 1.27)
+				)
+			)
+		)
+		(property "MPN" "2SK1958-VB"
+			(at 146.05 50.8 0)
+			(hide yes)
+			(show_name no)
+			(do_not_autoplace no)
+			(effects
+				(font
+					(size 1.27 1.27)
+				)
+			)
+		)
+		(property "LCSC Part" "C20755445"
+			(at 146.05 50.8 0)
+			(hide yes)

Commit message: cs: finalized KiCad files
Parts:
- Q15: value 2SK1958-VB -> 2N7002; LCSC Part C20755445 -> (none); MPN 2SK1958-VB -> (none)
Other:
- note added: "I_{max,Burst} = 7*(12V - 2V) / 1500Ω + 6*12V / 1000Ω = @{format( (7*(12 - 2) / 1500 + 6*12 / 1000) * 1000, 3)}mA I_{max,Cont} = 7*(12V - 2V) / 1500Ω + 6*12V / 11000Ω = @{format( (7*(12 - 2) / 1500 + 6*12 / 11000) * 1000, 3)}mA max Burst PD = R_{DS(on)} * I_{max,Burst}^{2} = @{format( 2 * (7*(12 - 2) / 1500 + 6*12 / 1000)^2 * 1000, 3)}mW @ R_{DS(on)}=2Ω max Cont. PD = R_{DS(on)} * I_{max,Cont}^{2}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"
- note added: "I_{max,Color} = (12V - 2V) / 1500Ω + 12V / 1000Ω = @{format(((12 - 2) / 1500 + 12 / 1000)* 1000, 3)}mA max PD = R_{DS(on)} * I_{max,Color}^{2} = @{format(( 2 * ((12 - 2) / 1500 + 12 / 1000)^2)*1000, 3)}mW @ R_{DS(on)}=2Ω max R_{DS(on)} = 200mW / (@{format(((12 - 2) / 1500 + 12 / 1000)* 1000, 3)}mA)^{2} = @{format(0.2 / ((12 - 2) / 1500 + 12 / 1000)^2, 0)}Ω"
- note removed: "max PD_{12V} = 12V * ((12V-2V)/1500ohm + 12V/1000ohm) = @{format(12 * ((12-2)/1500 + 12/1000), 3)}W max PD_{10V} = 10V * ((10V-2V)/1500ohm + 10V/1000ohm) = @{format(10 * ((10-2)/1500 + 10/1000), 3)}W"
- note removed: "max PD_{12V} = 12V * (7*(12V-2V)/1500ohm) + 6*12V/1000ohm) = @{format(12 * (7*(12-2)/1500 + 6*12/1000), 3)} W max PD_{10V} = 10V * (7*(10V-2V)/1500ohm) + 6*10V/1000ohm) = @{format(10 * (7*(10-2)/1500 + 6*10/1000), 3)} W"
Changed lines of the file:
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@@
 		)
 	)
-	(text "max PD_{12V} = 12V * (7*(12V-2V)/1500ohm) + 6*12V/1000ohm) = @{format(12 * (7*(12-2)/1500 + 6*12/1000), 3)} W\nmax PD_{10V} = 10V * (7*(10V-2V)/1500ohm) + 6*10V/1000ohm) = @{format(10 * (7*(10-2)/1500 + 6*10/1000), 3)} W\n"
+	(text "I_{max,Burst} = 7*(12V - 2V) / 1500Ω + 6*12V / 1000Ω = @{format( (7*(12 - 2) / 1500 + 6*12 / 1000) * 1000, 3)}mA\nI_{max,Cont} = 7*(12V - 2V) / 1500Ω + 6*12V / 11000Ω = @{format( (7*(12 - 2) / 1500 + 6*12 / 11000) * 1000, 3)}mA\n\nmax Burst PD = R_{DS(on)} * I_{max,Burst}^{2} = @{format( 2 * (7*(12 - 2) / 1500 + 6*12 / 1000)^2 * 1000, 3)}mW @ R_{DS(on)}=2Ω\nmax Cont. PD = R_{DS(on)} * I_{max,Cont}^{2} = @{format( 2 * (7*(12 - 2) / 1500 + 6*12 / 11000)^2 * 1000, 3)}mW @ R_{DS(on)}=2Ω\n"
 		(exclude_from_sim no)
-		(at 108.204 34.798 0)
+		(at 116.078 34.036 0)
 		(effects
 			(font
@@
 		)
 	)
-	(text "max PD_{12V} = 12V * ((12V-2V)/1500ohm + 12V/1000ohm) = @{format(12 * ((12-2)/1500 + 12/1000), 3)}W\nmax PD_{10V} = 10V * ((10V-2V)/1500ohm + 10V/1000ohm) = @{format(10 * ((10-2)/1500 + 10/1000), 3)}W"
+	(text "I_{max,Color} = (12V - 2V) / 1500Ω + 12V / 1000Ω = @{format(((12 - 2) / 1500 + 12 / 1000)* 1000, 3)}mA\nmax PD = R_{DS(on)} * I_{max,Color}^{2} = @{format(( 2 * ((12 - 2) / 1500 + 12 / 1000)^2)*1000, 3)}mW @ R_{DS(on)}=2Ω\nmax R_{DS(on)} = 200mW / (@{format(((12 - 2) / 1500 + 12 / 1000)* 1000, 3)}mA)^{2} = @{format(0.2 / ((12 - 2) / 1500 + 12 / 1000)^2, 0)}Ω"
 		(exclude_from_sim no)
 		(at 39.37 78.994 0)
@@
 	)
 	(symbol
+		(lib_id "Transistor_FET:2N7002")
+		(at 146.05 50.8 90)
+		(unit 1)
+		(body_style 1)
+		(exclude_from_sim no)
+		(in_bom yes)
+		(on_board yes)
+		(in_pos_files yes)
+		(dnp no)
+		(property "Reference" "Q15"
+			(at 146.05 42.164 90)
+			(show_name no)
+			(do_not_autoplace no)
+			(effects
+				(font
+					(size 1.27 1.27)
+				)
+			)
+		)
+		(property "Value" "2N7002"
+			(at 146.05 44.704 90)
+			(show_name no)
+			(do_not_autoplace no)
+			(effects
+				(font
+					(size 1.27 1.27)
+				)
+			)
+		)
+		(property "Footprint" "Package_TO_SOT_SMD:SOT-323_SC-70"
+			(at 147.955 45.72 0)
+			(hide yes)
+			(show_name no)
+			(do_not_autoplace no)
+			(effects
+				(font
+					(size 1.27 1.27)
+					(italic yes)
+				)
+				(justify left)
+			)
+		)
+		(property "Datasheet" "https://www.onsemi.com/pub/Collateral/NDS7002A-D.PDF"
+			(at 149.86 45.72 0)
+			(hide yes)
+			(show_name no)
+			(do_not_autoplace no)
+			(effects
+				(font
+					(size 1.27 1.27)
+				)
+				(justify left)
+			)
+		)
+		(property "Description" "0.115A Id, 60V Vds, N-Channel MOSFET, SOT-23"
+			(at 146.05 50.8 0)
+			(hide yes)
+			(show_name no)
+			(do_not_autoplace no)
+			(effects
+				(font
+					(size 1.27 1.27)
+				)
+			)
+		)
+		(property "Sim.Device" ""
+			(at 146.05 50.8 0)
+			(hide yes)
+			(show_name no)
+			(do_not_autoplace no)
+			(effects
+				(font
+					(size 1.27 1.27)
+				)
+			)
+		)
+		(pin "3"
+		)
+		(pin "1"
+		)
+		(pin "2"
+		)
+		(instances
+			(project "SLCU"
+				(path "/f738e776-c49a-4f35-8deb-cc918068af7e/1256c985-d505-4a7e-8bdd-0163862c50f7"
+					(reference "Q15")
+					(unit 1)
+				)
+			)
+		)
+	)
+	(symbol
 		(lib_id "PCM_Resistor_AKL:R_4x0603_Sep_Concave")
 		(at 60.96 138.43 180)
@@
 					(unit 1)
 				)
-			)
-		)
-	)
-	(symbol
-		(lib_id "Transistor_FET:2N7002")
-		(at 146.05 50.8 90)
-		(unit 1)
-		(body_style 1)
-		(exclude_from_sim no)
-		(in_bom yes)
-		(on_board yes)
-		(in_pos_files yes)
-		(dnp no)
-		(property "Reference" "Q15"
-			(at 146.05 42.164 90)
-			(show_name no)
-			(do_not_autoplace no)
-			(effects
-				(font
-					(size 1.27 1.27)
-				)
-			)
-		)
-		(property "Value" "2SK1958-VB"
-			(at 146.05 44.704 90)
-			(show_name no)
-			(do_not_autoplace no)
-			(effects
-				(font
-					(size 1.27 1.27)
-				)
-			)
-		)
-		(property "Footprint" "Package_TO_SOT_SMD:SOT-323_SC-70"
-			(at 147.955 45.72 0)
-			(hide yes)
-			(show_name no)
-			(do_not_autoplace no)
-			(effects
-				(font
-					(size 1.27 1.27)
-					(italic yes)
-				)
-				(justify left)
-			)
-		)
-		(property "Datasheet" "https://www.onsemi.com/pub/Collateral/NDS7002A-D.PDF"
-			(at 149.86 45.72 0)
-			(hide yes)
-			(show_name no)
-			(do_not_autoplace no)
-			(effects
-				(font
-					(size 1.27 1.27)
-				)
-				(justify left)
-			)
-		)
-		(property "Description" "0.115A Id, 60V Vds, N-Channel MOSFET, SOT-23"
-			(at 146.05 50.8 0)
-			(hide yes)
-			(show_name no)
-			(do_not_autoplace no)
-			(effects
-				(font
-					(size 1.27 1.27)
-				)
-			)
-		)
-		(property "Sim.Device" ""
-			(at 146.05 50.8 0)
-			(hide yes)
-			(show_name no)
-			(do_not_autoplace no)
-			(effects
-				(font
-					(size 1.27 1.27)
-				)
-			)
-		)
-		(property "MPN" "2SK1958-VB"
-			(at 146.05 50.8 0)
-			(hide yes)
-			(show_name no)
-			(do_not_autoplace no)
-			(effects
-				(font
-					(size 1.27 1.27)
-				)
-			)
-		)
-		(property "LCSC Part" "C20755445"
-			(at 146.05 50.8 0)
-			(hide yes)
-			(show_name no)
-			(do_not_autoplace no)
-			(effects
-				(font
-					(size 1.27 1.27)
-				)
-			)
-		)
-		(pin "3"
-		)
-		(pin "1"
-		)
-		(pin "2"
-		)
-		(instances
-			(project "SLCU"
-				(path "/f738e776-c49a-4f35-8deb-cc918068af7e/1256c985-d505-4a7e-8bdd-0163862c50f7"
-					(reference "Q15")
-					(unit 1)
-				)
