File: charging_station/KiCad/SLCU/LED_controller.kicad_sch (KiCad schematic)
At the start: 8 parts, among them Q18 2N7002, Q19 2N7002, Q20 2N7002, Q21 2N7002

Commit message: cs: corrected wrong mosfets on SLCU
Parts:
- Q19, Q20, Q21: value 2N7002 -> 2SK1958-VB; LCSC Part (none) -> C20755445; MPN (none) -> 2SK1958-VB
Other:
- note added: "max PD = 0.043 * (9.55 - 0.666) = @{format(0.043 * (9.55 - 0.666), 3)}W"
Changed lines of the file:
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@@
 		(title "SLCU (Stack Light Control Unit)")
 		(date "2026-10-10")
-		(rev "3.0")
+		(rev "3.1")
 		(company "JMU Würzburg")
 		(comment 1 "Nico Schubert")
@@
 			)
 			(justify left top)
+		)
+	)
+	(text "max PD = 0.043 * (9.55 - 0.666) = @{format(0.043 * (9.55 - 0.666), 3)}W"
+		(exclude_from_sim no)
+		(at 177.8 57.15 0)
+		(effects
+			(font
+				(size 1.27 1.27)
+			)
 		)
 	)
@@
 			)
 		)
-		(property "Value" "2N7002"
+		(property "Value" "2SK1958-VB"
 			(at 161.29 107.9499 0)
 			(show_name no)
@@
 		)
 		(property "Sim.Device" ""
+			(at 154.94 106.68 0)
+			(hide yes)
+			(show_name no)
+			(do_not_autoplace no)
+			(effects
+				(font
+					(size 1.27 1.27)
+				)
+			)
+		)
+		(property "MPN" "2SK1958-VB"
+			(at 154.94 106.68 0)
+			(hide yes)
+			(show_name no)
+			(do_not_autoplace no)
+			(effects
+				(font
+					(size 1.27 1.27)
+				)
+			)
+		)
+		(property "LCSC Part" "C20755445"
 			(at 154.94 106.68 0)
 			(hide yes)
@@
 			)
 		)
-		(property "Value" "2N7002"
+		(property "Value" "2SK1958-VB"
 			(at 181.61 76.1999 0)
 			(show_name no)
@@
 		)
 		(property "Sim.Device" ""
+			(at 175.26 74.93 0)
+			(hide yes)
+			(show_name no)
+			(do_not_autoplace no)
+			(effects
+				(font
+					(size 1.27 1.27)
+				)
+			)
+		)
+		(property "MPN" "2SK1958-VB"
+			(at 175.26 74.93 0)
+			(hide yes)
+			(show_name no)
+			(do_not_autoplace no)
+			(effects
+				(font
+					(size 1.27 1.27)
+				)
+			)
+		)
+		(property "LCSC Part" "C20755445"
 			(at 175.26 74.93 0)
 			(hide yes)
@@
 			)
 		)
-		(property "Value" "2N7002"
+		(property "Value" "2SK1958-VB"
 			(at 201.93 107.9499 0)
 			(show_name no)
@@
 			(at 195.58 106.68 0)
 			(hide yes)
+			(show_name no)
+			(do_not_autoplace no)
+			(effects
+				(font
+					(size 1.27 1.27)
+				)
+			)
+		)
+		(property "MPN" "2SK1958-VB"
+			(at 195.58 106.68 0)
+			(hide yes)
+			(show_name no)
+			(do_not_autoplace no)
+			(effects
+				(font
+					(size 1.27 1.27)
+				)
+			)
+		)
+		(property "LCSC Part" "C20755445"
+			(at 195.58 106.68 0)
+			(hide yes)

Commit message: cs: finalized KiCad files
Parts:
- Q19, Q20, Q21: value 2SK1958-VB -> 2N7002; LCSC Part C20755445 -> (none); MPN 2SK1958-VB -> (none)
Other:
- note added: "max PD = R_{DS(on)} * (0.043A)^{2} = @{format(2 * 0.043^2 * 1000, 0)}mW @ R_{DS(on)}=2Ω max R_{DS(on)} = 200mW / (50mA)^{2} = @{format(0.2 / (0.05)^2, 0)}Ω"
- note removed: "max PD = 0.043 * (9.55 - 0.666) = @{format(0.043 * (9.55 - 0.666), 3)}W"
