File: charging_station/KiCad/SLCU/power.kicad_sch (KiCad schematic)
At the start: 26 parts, among them Q1 AOI4185, U1 LMR51430

Commit message: cs: finalized KiCad files
Parts:
- R4: value 1.5k -> 3k
Changed lines of the file:
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@@
 				)
 			)
-			(table_cell "10"
+			(table_cell "12"
 				(exclude_from_sim no)
 				(at 200.66 99.06 0)
@@
 				)
 			)
-			(table_cell "47"
+			(table_cell "51"
 				(exclude_from_sim no)
 				(at 200.66 109.22 0)
@@
 			)
 		)
-		(property "Value" "1.5k"
+		(property "Value" "3k"
 			(at 210.82 35.5599 0)
 			(show_name no)
